File: PCB/RFC.kicad_pcb (KiCad board)
At the start: 4 copper layers, 100 x 40 mm, 71 parts, among them J1 Conn_01x01, J10 Conn_01x01, J11 Conn_01x01, J12 Conn_01x01, J13 Conn_01x01, J14 Conn_01x01, J15 Conn_01x01, J16 Conn_01x01, J17 Conn_01x01, J18 Conn_01x01, J19 Conn_01x01, J2 Conn_01x01, J20 Conn_01x01, J21 Conn_01x01, J22 Conn_01x01, J23 Conn_01x01, J24 Conn_01x01, J25 Conn_01x01, J26 Conn_01x01, J27 Conn_01x01, J28 Conn_01x01, J3 Conn_01x01, J4 Conn_01x01, J5 Conn_01x01, J6 Conn_01x01, J7 Conn_01x01, J8 Conn_01x01, J9 Conn_01x01, Q1 SI2302, SW1 SH-6X6X5H-TP, SW2 SH-6X6X5H-TP, U1 STM32F103C8Tx, U2 W25Q128JVS, U3 ICM-42688-P, U4 BMP388, U5 AP2112K-3.3TRG1, U6 219-2LPST, X1 3225-8.00-12-10-10/A

Commit message: renewed pcb
Parts:
- removed D2: LED_RAGB, LED_THT:LED_D5.0mm-4_RGB
- removed R5, R6, R7: 1KΩ (1001) ±1%, lcsc_footprints:C22548_R0603
- added D4: LED_RAGB, LED_THT:LED_D5.0mm-4_RGB, F.Cu at (145.3, -304.0)
- added R10: 1KΩ (1001) ±1%, lcsc_footprints:C22548_R0603, F.Cu at (137.7, -301.5)
- added R11: 1KΩ (1001) ±1%, lcsc_footprints:C22548_R0603, F.Cu at (137.7, -304.0)
- added R12: 1KΩ (1001) ±1%, lcsc_footprints:C22548_R0603, F.Cu at (137.7, -306.4)
Connections:
- net Net-(J3-Pin_1) renamed /PYROARM
- net Net-(J4-Pin_1) renamed /ARM
- net Net-(J5-Pin_1) renamed /SERVO1
- net Net-(J6-Pin_1) renamed /SERVO2
- net Net-(J7-Pin_1) renamed /SERVO3
- net Net-(J8-Pin_1) renamed /SERVO4
- net Net-(U1-BOOT0) renamed /BOOT0
- net Net-(U1-NRST) renamed /NRST
- net Net-(U1-PA10) renamed /FLASHCS
- net Net-(U1-PA12) renamed /TEST
- net Net-(U1-PA13) renamed /SWDIO
- net Net-(U1-PA14) renamed /SWCLK
- net Net-(U1-PA5) renamed /SCK
- net Net-(U1-PA6) renamed /MISO
- net Net-(U1-PA7) renamed /MOSI
- net Net-(U1-PA8) renamed /BMPCS
- net Net-(U1-PA9) renamed /IMUCS
- net Net-(U1-PB1) renamed /BATTSENSE
- net Net-(U1-PB9) renamed /BUZZER
- net Net-(U1-PD0) renamed /OSC_IN
- net Net-(U1-PD1) renamed /OSC_OUT
- C1 pad 1: Net-(U3-VDDIO) -> +3.3V
- C2 pad 1: Net-(U3-VDD) -> +3.3V
- C3 pad 1: Net-(U3-VDD) -> +3.3V
- D1 pad 1: +3.3V -> Net-(D1-C)
- D1 pad 2: Net-(D1-A) -> +3.3V
- H1 pad 1: +3.3V -> +3V3
- H2 pad 1: +3.3V -> +3V3
- H2 pad 3: Net-(U1-PB11) -> /USART3_TX
- H2 pad 4: Net-(U1-PB10) -> /USART3_RX
- H3 pad 3: Net-(U1-PB11) -> /USART3_TX
- H3 pad 4: Net-(U1-PB10) -> /USART3_RX
- J11 pad 1: +3.3V -> Net-(D1-C)
- J12 pad 1: Net-(D1-A) -> +3.3V
- Q1 pad 3: Net-(D1-A) -> +3.3V
- R1 pad 1: +3.3V -> 3V3
- U1 pad 18: Net-(U1-PB0) -> /R
- U1 pad 20: Net-(U1-PB2) -> /G
- U1 pad 21: Net-(U1-PB10) -> /USART3_TX
- U1 pad 22: Net-(U1-PB11) -> /USART3_RX
- U1 pad 25: unconnected-(U1-PB12-Pad25) -> /PyroCont1
- U1 pad 26: unconnected-(U1-PB13-Pad26) -> /PyroCont2
- U1 pad 39: Net-(U1-PB3) -> /B
- U1 pad 41: unconnected-(U1-PB5-Pad41) -> /Pyro1
- U1 pad 42: unconnected-(U1-PB6-Pad42) -> /Pyro2
- U2 pad 3: +3.3V -> +3V3
- U2 pad 7: +3.3V -> +3V3
- U3 pad 5: Net-(U3-VDDIO) -> +3.3V
- U3 pad 8: Net-(U3-VDD) -> +3.3V
