File: PCB/RFC.kicad_sch (KiCad schematic)
At the start: 67 parts, among them J1 Conn_01x01, J10 Conn_01x01, J11 Conn_01x01, J12 Conn_01x01, J13 Conn_01x01, J14 Conn_01x01, J15 Conn_01x01, J16 Conn_01x01, J17 Conn_01x01, J18 Conn_01x01, J19 Conn_01x01, J2 Conn_01x01, J20 Conn_01x01, J21 Conn_01x01, J22 Conn_01x01, J23 Conn_01x01, J24 Conn_01x01, J25 Conn_01x01, J26 Conn_01x01, J27 Conn_01x01, J28 Conn_01x01, J3 Conn_01x01, J4 Conn_01x01, J5 Conn_01x01, J6 Conn_01x01, J7 Conn_01x01, J8 Conn_01x01, J9 Conn_01x01, Q1 SI2302, SW1 SH-6X6X5H-TP, SW2 SH-6X6X5H-TP, U1 STM32F103C8Tx, U2 W25Q128JVS, U3 ICM-42688-P, U4 BMP388, U5 AP2112K-3.3TRG1, U6 219-2LPST, X1 3225-8.00-12-10-10/A

Commit message: renewed pcb
Parts:
- removed D2: LED_RAGB, LED_THT:LED_D5.0mm-4_RGB, symbol Device:LED_RAGB
- removed J23, J24, J27, J28: Conn_01x01, Connector_Wire:SolderWire-1sqmm_1x01_D1.4mm_OD2.7mm, symbol Connector_Generic:Conn_01x01
- removed R5, R6, R7: 1KΩ (1001) ±1%, lcsc_footprints:C22548_R0603, symbol MAIN:1KΩ_(1001)_±1%
- added D4: LED_RAGB, LED_THT:LED_D5.0mm-4_RGB, symbol Device:LED_RAGB
- added J29, J30: Conn_01x02, symbol Connector_Generic:Conn_01x02
- added R10, R11, R12: 1KΩ (1001) ±1%, lcsc_footprints:C22548_R0603, symbol MAIN:1KΩ_(1001)_±1%
Connections:
- net +3.3V: now also C1.1, C2.1, C3.1, D1.2 (A), J12.1 (Pin_1), Q1.3 (D), U3.5 (VDDIO), U3.8 (VDD); no longer D1.1 (C), H1.1, H2.1, J11.1 (Pin_1), R1.1, U2.3 (~{WP}/IO_{2}), U2.7 (~{HOLD}/~{RESET}/IO_{3})
- net USART3_TX: now reaches H2.3, H3.3
- net USART3_TX: now also U1.21 (PB10); no longer U1.22 (PB11)
- net USART3_RX: now reaches H2.4, H3.4
- net USART3_RX: now also U1.22 (PB11); no longer U1.21 (PB10)
- net BATTSENSE: now reaches R3.2, R4.2, U1.19 (PB1)
- net NRST: now reaches H1.5, R1.2, SW2.4, U1.7 (NRST)
- net G: now reaches U1.20 (PB2)
- net G: now also R11.2
- net MISO: now reaches U1.16 (PA6), U2.2 (DO/IO_{1}), U3.1 (AP_SDO/AP_AD0), U4.5 (SDO)
- net IMUCS: now reaches U1.30 (PA9), U3.12 (AP_CS)
- net SCK: now reaches U1.15 (PA5), U2.6 (CLK), U3.13 (AP_SCL/AP_SCLK), U4.2 (SCK)
- net MOSI: now reaches U1.17 (PA7), U2.5 (DI/IO_{0}), U3.14 (AP_SDA/AP_SDIO/AP_SDI), U4.4 (SDI)
- net OSC_IN: now reaches C4.1, U1.5 (PD0), X1.1
- net SERVO4: now reaches J8.1 (Pin_1), U1.13 (PA3)
- net TEST: now reaches U1.33 (PA12), U6.2
- net ARM: now reaches J4.1 (Pin_1), U1.32 (PA11)
- net BUZZER: now reaches R9.1, U1.46 (PB9)
- net R: now reaches U1.18 (PB0)
- net R: now also R10.2
- net PYROARM: now reaches J3.1 (Pin_1), U1.38 (PA15)
- net OSC_OUT: now reaches C5.1, U1.6 (PD1), X1.3
- net BOOT0: now reaches R2.2, SW1.4, U1.44 (BOOT0)
- net SERVO2: now reaches J6.1 (Pin_1), U1.11 (PA1)
- net SERVO3: now reaches J7.1 (Pin_1), U1.12 (PA2)
- net SERVO1: now reaches J5.1 (Pin_1), U1.10 (PA0)
- net BMPCS: now reaches U1.29 (PA8), U4.6 (CSB)
- net B: now reaches U1.39 (PB3)
- net B: now also R12.2
- net SWDIO: now reaches H1.3, U1.34 (PA13)
- net SWCLK: now reaches H1.4, U1.37 (PA14)
- net FLASHCS: now reaches U1.31 (PA10), U2.1 (~{CS})
- net PyroCont1: now reaches U1.25 (PB12)
- net PyroCont1: now also J30.2 (Pin_2)
- net PyroCont2: now reaches U1.26 (PB13)
- net PyroCont2: now also J30.1 (Pin_1)
- net Pyro1: now reaches U1.41 (PB5)
- net Pyro1: now also J29.2 (Pin_2)
- net Pyro2: now reaches U1.42 (PB6)
- net Pyro2: now also J29.1 (Pin_1)
- new net: D4.4 (BK), R12.1
- new net: D1.1 (C), J11.1 (Pin_1)
- new net: D4.3 (GK), R11.1
- new net: D4.1 (RK), R10.1
- new net +3V3: H1.1, H2.1, U2.3 (~{WP}/IO_{2}), U2.7 (~{HOLD}/~{RESET}/IO_{3})
- new net 3V3: R1.1
- no-connect marks 15 -> 20
Other:
- moved on the sheet: C1, C10, C11, C12, C13, C14, C2, C3, C4, C5, C6, C7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
